Commit message: summit_x_description: added correct position for the asus xtion camera

File: summit_x_description/robots/summit_x.urdf.xacro (robot description, xacro)
@@ -80,4 +80,7 @@
 	</xacro:sensor_kinect>
 -->
+	<xacro:sensor_asus_xtion_pro name="xtion_pro" parent="rover_link">
+		<origin xyz="0.13 0.0 0.1" rpy="0 0 0"/>
+	</xacro:sensor_asus_xtion_pro>
 <!--
 	<xacro:sensor_fotonic name="fotonic" parent="base_link">

File: summit_x_description/urdf/bases/summit_x_base.urdf.xacro (robot description, xacro)
@@ -91,4 +91,5 @@
 	 </actuator>
   </transmission>
+<!--
 	<joint name="camera_joint" type="fixed">
 			<axis xyz="0 1 0" />
@@ -105,5 +106,7 @@
 		</inertial>
 	</link>
+-->
   <!-- Axis camera properties-->
+<!--
 	<xacro:property name="ptz_joint_effort_limit" value="100.0" />
   <xacro:property name="ptz_joint_velocity_limit" value="100.0"/>
@@ -111,4 +114,5 @@
   <xacro:property name="ptz_joint_damping" value="0.1" />
   <xacro:property name="ptz_mechanical_reduction" value="1.0" />
+-->
 <!--
   <joint name="joint_camera_pan" type="continuous">
