Commit message: Fixed hardware interface

File: summit_x_description/urdf/bases/summit_x_base.urdf.xacro (robot description, xacro)
@@ -84,10 +84,11 @@
   </joint>
   <transmission name="joint_scissor_trans">
-	 <type>transmission_interface/SimpleTransmission</type>
-     <joint name="scissor_prismatic_joint" />
-     <actuator name="scissor_motor">
-		<hardwareInterface>EffortJointInterface</hardwareInterface>
-		<mechanicalReduction>1</mechanicalReduction>
-	 </actuator>
+    <type>transmission_interface/SimpleTransmission</type>
+    <joint name="scissor_prismatic_joint">
+      <hardwareInterface>EffortJointInterface</hardwareInterface>
+    </joint>
+    <actuator name="scissor_motor">
+      <mechanicalReduction>1</mechanicalReduction>
+     </actuator>
   </transmission>
 <!--

File: summit_x_description/urdf/wheels/omni_wheel.urdf.xacro (robot description, xacro)
@@ -71,7 +71,8 @@
     <transmission name="${name}_wheel_joint_trans">
       <type>transmission_interface/SimpleTransmission</type>
-      <joint name="joint_${name}_wheel" />
+      <joint name="joint_${name}_wheel">
+        <hardwareInterface>EffortJointInterface</hardwareInterface>
+      </joint>
       <actuator name="${name}_wheel_joint_motor">
-        <hardwareInterface>EffortJointInterface</hardwareInterface>
         <mechanicalReduction>1</mechanicalReduction>
       </actuator>

File: summit_x_description/urdf/wheels/rubber_wheel.urdf.xacro (robot description, xacro)
@@ -58,7 +58,8 @@
     <transmission name="${name}_wheel_joint_trans">
       <type>transmission_interface/SimpleTransmission</type>
-      <joint name="joint_${name}_wheel" />
+      <joint name="joint_${name}_wheel">
+        <hardwareInterface>EffortJointInterface</hardwareInterface>
+      </joint>
       <actuator name="${name}_wheel_joint_motor">
-        <hardwareInterface>EffortJointInterface</hardwareInterface>
         <mechanicalReduction>1</mechanicalReduction>
       </actuator>
